File: iobbq_main.brd (EAGLE design)
At the start: 100 x 100 mm, 100 parts, among them K1 SRD-5VDC-SL-C, K2 SRD-5VDC-SL-C, X1 JST-XH-5-B5B-XH-A, X10 MPT0.5/8-2.54, X11 PIIKKIRIMA-7, X12 TE_RUUVULIITIN2, X13 TE_RUUVILIITIN2, X14 TE_RUUVILIITIN2, X16 TE_RUUVILIITIN3, X2 MPT0.5/8-2.54, X3 JST-XH-5-B5B-XH-A, X4 MPT0.5/8-2.54, X5 MPT0.5/8-2.54, X6 MPT0.5/8-2.54, X7 MPT0.5/8-2.54, X8 PIIKKIRIMA-4, X9 PIIKKIRIMA-7

Commit message: update values
Parts:
- added U$3: DAFUG, dafug:DAFUG
- C1, C12, C2, C26, C3: value CAP0603 -> 100n
- C10, C11: value CAP0805 -> 10µ 16V
- C13, C24, C25, C4, C5, C6, C7, C8, C9: value CAP0805 -> 1µ 16V
- C18: value CAP0805 -> 10n
- C19, C20: value CAP0603 -> NA
- C21, C22: value CAP0805 -> 2µ2 50V
- D1, D9: value (none) -> STPS340U
- N2: value LD117AS33TR -> AZ1117EH-3.3
- OK1, OK2, OK3, OK4, OK5, OK6: value SFH6186-2 -> EL817SC
- R1: value RES0603 -> 402R 0.1%
- R10, R11, R12, R13, R14, R15, R16, R17, R18, R19, R2, R20, R21, R22, R23, R24, R25, R26, R27, R28, R39, R43, R44, R45, R9: value RES0603 -> 3k24
- R3, R4, R5, R6, R7, R8: value RES0805 -> 1k21
- R38: value RES0603 -> 10k0
- R40: value RES0603 -> NA
- X12: value TE_RUUVULIITIN2 -> TE 282837-2
- X13, X14: value TE_RUUVILIITIN2 -> TE 282837-2
- X16: value TE_RUUVILIITIN3 -> TE 282837-3

Commit message: pull ESP8266 GPIO15 down
Parts:
- added R29: 3k24, OMAT_IC:R0603
Connections:
- new net N$17: A1.10, R29.2
- net GND: now also R29.1
Routing:
- net N$17: track 0.00 -> 10.3 mm
Changed lines of the file:
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@@
 <setting verticaltext="up"/>
 </settings>
-<grid distance="0.25" unitdist="mm" unit="mm" style="lines" multiple="1" display="no" altdistance="0.025" altunitdist="inch" altunit="inch"/>
+<grid distance="0.1" unitdist="mm" unit="mm" style="lines" multiple="1" display="no" altdistance="0.025" altunitdist="inch" altunit="inch"/>
 <layers>
 <layer number="1" name="Top" color="4" fill="1" visible="yes" active="yes"/>
@@
 <element name="U$1" library="dafug" package="DAFUG" value="" x="89.75" y="9" rot="MR0"/>
 <element name="U$3" library="dafug" package="DAFUG" value="DAFUG" x="-2.75" y="2.5"/>
+<element name="R29" library="OMAT_IC" package="R0603" value="3k24" x="85.25" y="75.25" smashed="yes" rot="R180">
+<attribute name="NAME" x="87.085" y="74.315" size="1.2" layer="25" font="vector" rot="R180"/>
+<attribute name="VALUE" x="85.885" y="77.155" size="0.8128" layer="27" rot="R180"/>
+</element>
 </elements>
 <signals>
@@
 <via x="28.6" y="69.25" extent="1-16" drill="0.4"/>
 <via x="15.1" y="77" extent="1-16" drill="1"/>
+<contactref element="R29" pad="1"/>
 </signal>
 <signal name="+5V">
@@
 <wire x1="95.84" y1="81.25" x2="96" y2="81.09" width="0.25" layer="1"/>
 </signal>
+<signal name="N$17">
+<contactref element="R29" pad="2"/>
+<contactref element="A1" pad="10"/>
+<wire x1="84.525" y1="75.25" x2="84.525" y2="80.425" width="0.4" layer="1"/>
+<wire x1="84.525" y1="80.425" x2="85.9" y2="81.8" width="0.4" layer="1"/>
+<wire x1="85.9" y1="81.8" x2="89.07" y2="81.8" width="0.4" layer="1"/>
+<wire x1="89.07" y1="81.8" x2="89.09" y2="81.78" width="0.4" layer="1"/>
+</signal>
 </signals>
